Commit message: update launchfiles and configs files for current version of snp

File: urdf/workcell.xacro (robot description, xacro)
@@ -3,4 +3,6 @@
   <xacro:include filename="$(find motoman_hc10_support)/urdf/hc10dt_macro.xacro" />
   <xacro:motoman_hc10dt prefix=""/>
+  <xacro:include filename="$(find snp_automate_2023)/urdf/ros2_control.xacro"/>
+  <xacro:snp_ros2_control name="SNP ROS2 Control" prefix=""/>
   <xacro:property name="dt_flange_width" value="0.040"/>
   <!-- Add World -->
@@ -163,5 +165,5 @@
     <origin rpy="0.0 0.0 ${radians(45)}"/>
   </joint>
-  <xacro:property name="camera_cal" value="${load_yaml('$(find snp_automate_2023)/config/calibration.yaml')}" />
+  <xacro:property name="camera_cal" value="${xacro.load_yaml('$(find snp_automate_2023)/config/calibration.yaml')}" />
   <link name="camera_color_optical_frame"/>
   <joint name="tool0_to_camera" type="fixed">
