Commit message: Updated URDF

File: snp_automate_2023/urdf/workcell.xacro (robot description, xacro)
@@ -38,5 +38,5 @@
     <visual>
       <geometry>
-        <mesh filename="package://snp_automate_2023/meshes/visual/steel_table.ply"/>
+        <mesh filename="package://snp_support/meshes/steel_table.ply"/>
       </geometry>
       <material name="dark_gray"/>
@@ -44,5 +44,5 @@
     <collision>
       <geometry>
-        <mesh filename="package://snp_automate_2023/meshes/collision/steel_table.ply"/>
+        <mesh filename="package://snp_support/meshes/steel_table.ply"/>
       </geometry>
     </collision>
@@ -71,55 +71,79 @@
   </joint>
   <!-- Add End Effector Components -->
+  <xacro:property name="radius" value="${3.75 * 0.0254 / 2.0}"/>
+  <xacro:property name="length" value="${5.875 * 0.0254}"/>
+  <xacro:property name="small_radius" value="${1.0 * 0.0254 / 2.0}"/>
+  <xacro:property name="small_length" value="${2.0 * 0.0254}"/>
   <link name="ee">
     <visual>
       <geometry>
-        <mesh filename="package://snp_automate_2023/meshes/visual/end_effector.stl"/>
+        <mesh filename="package://snp_support/meshes/ati_spindle.ply"/>
       </geometry>
     </visual>
-    <collision name="compliance">
+    <visual>
       <geometry>
-        <mesh filename="package://snp_automate_2023/meshes/collision/afd310.ply"/>
+        <mesh filename="package://snp_support/meshes/ati_hose.ply"/>
+      </geometry>
+    </visual>
+    <visual>
+      <geometry>
+        <mesh filename="package://snp_support/meshes/ati_tool.ply"/>
+      </geometry>
+    </visual>
+    <visual>
+      <geometry>
+        <mesh filename="package://snp_support/meshes/ati_bracket.ply"/>
+      </geometry>
+    </visual>
+    <visual>
+      <geometry>
+        <mesh filename="package://snp_support/meshes/ati_standoff.ply"/>
+      </geometry>
+    </visual>
+    <visual>
+      <geometry>
+        <mesh filename="package://snp_support/meshes/hc10_standoff.ply"/>
+      </geometry>
+    </visual>
+    <visual>
+      <geometry>
+        <mesh filename="package://snp_support/meshes/sensor_bracket.ply"/>
+      </geometry>
+    </visual>
+    <!-- Collision -->
+    <collision>
+      <geometry>
+        <mesh filename="package://snp_support/meshes/ati_spindle.ply"/>
       </geometry>
     </collision>
-    <collision name="spindle">
+    <collision>
       <geometry>
-        <mesh filename="package://snp_automate_2023/meshes/collision/rps100.ply"/>
+        <mesh filename="package://snp_support/meshes/ati_hose.ply"/>
       </geometry>
     </collision>
-    <collision name="backplate">
+    <collision>
       <geometry>
-        <mesh filename="package://snp_automate_2023/meshes/collision/backplate.ply"/>
+        <mesh filename="package://snp_support/meshes/ati_tool.ply"/>
       </geometry>
     </collision>
-    <collision name="frontplate">
+    <collision>
       <geometry>
-        <mesh filename="package://snp_automate_2023/meshes/collision/front.ply"/>
+        <mesh filename="package://snp_support/meshes/ati_bracket.ply"/>
       </geometry>
     </collision>
-    <collision name="camera1">
+    <collision>
       <geometry>
-        <mesh filename="package://snp_automate_2023/meshes/collision/camera1.ply"/>
+        <mesh filename="package://snp_support/meshes/ati_standoff.ply"/>
       </geometry>
     </collision>
-    <collision name="camera2">
+    <collision>
       <geometry>
-        <mesh filename="package://snp_automate_2023/meshes/collision/camera2.ply"/>
+        <mesh filename="package://snp_support/meshes/hc10_standoff.ply"/>
       </geometry>
     </collision>
-    <collision name="sidebracket1">
+    <collision>
       <geometry>
-        <mesh filename="package://snp_automate_2023/meshes/collision/bracket1.ply"/>
+        <mesh filename="package://snp_support/meshes/sensor_bracket.ply"/>
       </geometry>
-    </collision>
-    <collision name="sidebracket2">
-      <geometry>
-        <mesh filename="package://snp_automate_2023/meshes/collision/bracket2.ply"/>
-      </geometry>
-    </collision>
-    <collision name="tcp">
-      <geometry>
-        <cylinder radius="${1.5 * 0.0254}" length="${2.0 * 0.0254}"/>
-      </geometry>
-      <origin xyz="${-0.263 + 1.5 * 0.0254} 0.0 0.083" rpy="0 ${radians(-90)} 0"/>
     </collision>
   </link>
@@ -128,5 +152,5 @@
     <child link="ee"/>
   </joint>
-  <xacro:property name="camera_cal" value="${load_yaml('$(find snp_automate_2023)/config/camera_calibration.yaml')}" />
+  <xacro:property name="camera_cal" value="${load_yaml('$(find snp_support)/config/camera_calibration.yaml')}" />
   <link name="camera_color_optical_frame"/>
   <joint name="tool0_to_camera" type="fixed">
@@ -148,5 +172,5 @@
     <parent link="tool_flange"/>
     <child link="sand_tcp"/>
-    <origin xyz="-0.26261 0 ${0.08259 + dt_flange_width}" rpy="${radians(-90)} 0 ${radians(90)}"/>
+    <origin xyz="-0.186 0.0 ${0.08325 + dt_flange_width}" rpy="0.0 ${radians(90)} 0.0"/>
   </joint>
 </robot>

Commit message: Updated URDF

File: snp_automate_2023/urdf/workcell.xacro (robot description, xacro)
@@ -38,5 +38,5 @@
     <visual>
       <geometry>
-        <mesh filename="package://snp_support/meshes/steel_table.ply"/>
+        <mesh filename="package://snp_automate_2023/meshes/steel_table.ply"/>
       </geometry>
       <material name="dark_gray"/>
@@ -44,5 +44,5 @@
     <collision>
       <geometry>
-        <mesh filename="package://snp_support/meshes/steel_table.ply"/>
+        <mesh filename="package://snp_automate_2023/meshes/steel_table.ply"/>
       </geometry>
     </collision>
@@ -78,35 +78,35 @@
     <visual>
       <geometry>
-        <mesh filename="package://snp_support/meshes/ati_spindle.ply"/>
+        <mesh filename="package://snp_automate_2023/meshes/ati_spindle.ply"/>
       </geometry>
     </visual>
     <visual>
       <geometry>
-        <mesh filename="package://snp_support/meshes/ati_hose.ply"/>
+        <mesh filename="package://snp_automate_2023/meshes/ati_hose.ply"/>
       </geometry>
     </visual>
     <visual>
       <geometry>
-        <mesh filename="package://snp_support/meshes/ati_tool.ply"/>
+        <mesh filename="package://snp_automate_2023/meshes/ati_tool.ply"/>
       </geometry>
     </visual>
     <visual>
       <geometry>
-        <mesh filename="package://snp_support/meshes/ati_bracket.ply"/>
+        <mesh filename="package://snp_automate_2023/meshes/ati_bracket.ply"/>
       </geometry>
     </visual>
     <visual>
       <geometry>
-        <mesh filename="package://snp_support/meshes/ati_standoff.ply"/>
+        <mesh filename="package://snp_automate_2023/meshes/ati_standoff.ply"/>
       </geometry>
     </visual>
     <visual>
       <geometry>
-        <mesh filename="package://snp_support/meshes/hc10_standoff.ply"/>
+        <mesh filename="package://snp_automate_2023/meshes/hc10_standoff.ply"/>
       </geometry>
     </visual>
     <visual>
       <geometry>
-        <mesh filename="package://snp_support/meshes/sensor_bracket.ply"/>
+        <mesh filename="package://snp_automate_2023/meshes/sensor_bracket.ply"/>
       </geometry>
     </visual>
@@ -114,35 +114,35 @@
     <collision>
       <geometry>
-        <mesh filename="package://snp_support/meshes/ati_spindle.ply"/>
+        <mesh filename="package://snp_automate_2023/meshes/ati_spindle.ply"/>
       </geometry>
     </collision>
     <collision>
       <geometry>
-        <mesh filename="package://snp_support/meshes/ati_hose.ply"/>
+        <mesh filename="package://snp_automate_2023/meshes/ati_hose.ply"/>
       </geometry>
     </collision>
     <collision>
       <geometry>
-        <mesh filename="package://snp_support/meshes/ati_tool.ply"/>
+        <mesh filename="package://snp_automate_2023/meshes/ati_tool.ply"/>
       </geometry>
     </collision>
     <collision>
       <geometry>
-        <mesh filename="package://snp_support/meshes/ati_bracket.ply"/>
+        <mesh filename="package://snp_automate_2023/meshes/ati_bracket.ply"/>
       </geometry>
     </collision>
     <collision>
       <geometry>
-        <mesh filename="package://snp_support/meshes/ati_standoff.ply"/>
+        <mesh filename="package://snp_automate_2023/meshes/ati_standoff.ply"/>
       </geometry>
     </collision>
     <collision>
       <geometry>
-        <mesh filename="package://snp_support/meshes/hc10_standoff.ply"/>
+        <mesh filename="package://snp_automate_2023/meshes/hc10_standoff.ply"/>
       </geometry>
     </collision>
     <collision>
       <geometry>
-        <mesh filename="package://snp_support/meshes/sensor_bracket.ply"/>
+        <mesh filename="package://snp_automate_2023/meshes/sensor_bracket.ply"/>
       </geometry>
     </collision>
@@ -152,5 +152,5 @@
     <child link="ee"/>
   </joint>
-  <xacro:property name="camera_cal" value="${load_yaml('$(find snp_support)/config/camera_calibration.yaml')}" />
+  <xacro:property name="camera_cal" value="${load_yaml('$(find snp_automate_2023)/config/camera_calibration.yaml')}" />
   <link name="camera_color_optical_frame"/>
   <joint name="tool0_to_camera" type="fixed">

Commit message: Updated calibration; changed file name

File: snp_automate_2023/urdf/workcell.xacro (robot description, xacro)
@@ -151,6 +151,7 @@
     <parent link="tool0"/>
     <child link="ee"/>
+    <origin rpy="0.0 0.0 ${radians(45)}"/>
   </joint>
-  <xacro:property name="camera_cal" value="${load_yaml('$(find snp_automate_2023)/config/camera_calibration.yaml')}" />
+  <xacro:property name="camera_cal" value="${load_yaml('$(find snp_automate_2023)/config/calibration.yaml')}" />
   <link name="camera_color_optical_frame"/>
   <joint name="tool0_to_camera" type="fixed">

Commit message: Updated TCP location; added half sphere to end effector geometry

File: snp_automate_2023/urdf/workcell.xacro (robot description, xacro)
@@ -111,4 +111,9 @@
       </geometry>
     </visual>
+    <visual>
+      <geometry>
+        <mesh filename="package://snp_automate_2023/meshes/sponge.ply"/>
+      </geometry>
+    </visual>
     <!-- Collision -->
     <collision>
@@ -147,4 +152,9 @@
       </geometry>
     </collision>
+    <collision>
+      <geometry>
+        <mesh filename="package://snp_automate_2023/meshes/sponge.ply"/>
+      </geometry>
+    </collision>
   </link>
   <joint name="tool0_to_ee" type="fixed">
@@ -172,6 +182,9 @@
   <joint name="sand_tcp_joint" type="fixed">
     <parent link="tool_flange"/>
+<!--    <origin xyz="-0.158 -0.158 0.123" rpy="0.0 ${radians(90)} ${radians(-135)}"/>-->
+    <origin xyz="-0.149 -0.149 0.123" rpy="0.0 ${radians(90)} ${radians(-135)}"/>
+<!--    <parent link="ee"/>-->
+<!--    <origin xyz="${-0.186 - 0.038} 0.0 ${0.08325}" rpy="0.0 ${radians(90)} 0.0"/>-->
     <child link="sand_tcp"/>
-    <origin xyz="-0.186 0.0 ${0.08325 + dt_flange_width}" rpy="0.0 ${radians(90)} 0.0"/>
   </joint>
 </robot>

Commit message: increase min z tsdf and tcp frame offset

File: snp_automate_2023/urdf/workcell.xacro (robot description, xacro)
@@ -185,5 +185,5 @@
     <parent link="tool_flange"/>
 <!--    <origin xyz="-0.158 -0.158 0.123" rpy="0.0 ${radians(90)} ${radians(-135)}"/>-->
-    <origin xyz="-0.149 -0.149 0.123" rpy="0.0 ${radians(90)} ${radians(-135)}"/>
+    <origin xyz="-0.149 ${-0.149 - 0.005} 0.123" rpy="0.0 ${radians(90)} ${radians(-135)}"/>
 <!--    <parent link="ee"/>-->
 <!--    <origin xyz="${-0.186 - 0.038} 0.0 ${0.08325}" rpy="0.0 ${radians(90)} 0.0"/>-->

Commit message: add visual mesh for table

File: snp_automate_2023/urdf/workcell.xacro (robot description, xacro)
@@ -40,5 +40,5 @@
     <visual>
       <geometry>
-        <mesh filename="package://snp_automate_2023/meshes/steel_table.ply"/>
+        <mesh filename="package://snp_automate_2023/meshes/visual/steel_table.ply"/>
       </geometry>
       <material name="dark_gray"/>
@@ -46,5 +46,5 @@
     <collision>
       <geometry>
-        <mesh filename="package://snp_automate_2023/meshes/steel_table.ply"/>
+        <mesh filename="package://snp_automate_2023/meshes/collision/steel_table.ply"/>
       </geometry>
     </collision>
@@ -80,40 +80,40 @@
     <visual>
       <geometry>
-        <mesh filename="package://snp_automate_2023/meshes/ati_spindle.ply"/>
+        <mesh filename="package://snp_automate_2023/meshes/collision/ati_spindle.ply"/>
       </geometry>
     </visual>
     <visual>
       <geometry>
-        <mesh filename="package://snp_automate_2023/meshes/ati_hose.ply"/>
+        <mesh filename="package://snp_automate_2023/meshes/collision/ati_hose.ply"/>
       </geometry>
     </visual>
     <visual>
       <geometry>
-        <mesh filename="package://snp_automate_2023/meshes/ati_tool.ply"/>
+        <mesh filename="package://snp_automate_2023/meshes/collision/ati_tool.ply"/>
       </geometry>
     </visual>
     <visual>
       <geometry>
-        <mesh filename="package://snp_automate_2023/meshes/ati_bracket.ply"/>
+        <mesh filename="package://snp_automate_2023/meshes/collision/ati_bracket.ply"/>
       </geometry>
     </visual>
     <visual>
       <geometry>
-        <mesh filename="package://snp_automate_2023/meshes/ati_standoff.ply"/>
+        <mesh filename="package://snp_automate_2023/meshes/collision/ati_standoff.ply"/>
       </geometry>
     </visual>
     <visual>
       <geometry>
-        <mesh filename="package://snp_automate_2023/meshes/hc10_standoff.ply"/>
+        <mesh filename="package://snp_automate_2023/meshes/collision/hc10_standoff.ply"/>
       </geometry>
     </visual>
     <visual>
       <geometry>
-        <mesh filename="package://snp_automate_2023/meshes/sensor_bracket.ply"/>
+        <mesh filename="package://snp_automate_2023/meshes/collision/sensor_bracket.ply"/>
       </geometry>
     </visual>
     <visual>
       <geometry>
-        <mesh filename="package://snp_automate_2023/meshes/sponge.ply"/>
+        <mesh filename="package://snp_automate_2023/meshes/collision/sponge.ply"/>
       </geometry>
     </visual>
@@ -121,40 +121,40 @@
     <collision>
       <geometry>
-        <mesh filename="package://snp_automate_2023/meshes/ati_spindle.ply"/>
+        <mesh filename="package://snp_automate_2023/meshes/collision/ati_spindle.ply"/>
       </geometry>
     </collision>
     <collision>
       <geometry>
-        <mesh filename="package://snp_automate_2023/meshes/ati_hose.ply"/>
+        <mesh filename="package://snp_automate_2023/meshes/collision/ati_hose.ply"/>
       </geometry>
     </collision>
     <collision>
       <geometry>
-        <mesh filename="package://snp_automate_2023/meshes/ati_tool.ply"/>
+        <mesh filename="package://snp_automate_2023/meshes/collision/ati_tool.ply"/>
       </geometry>
     </collision>
     <collision>
       <geometry>
-        <mesh filename="package://snp_automate_2023/meshes/ati_bracket.ply"/>
+        <mesh filename="package://snp_automate_2023/meshes/collision/ati_bracket.ply"/>
       </geometry>
     </collision>
     <collision>
       <geometry>
-        <mesh filename="package://snp_automate_2023/meshes/ati_standoff.ply"/>
+        <mesh filename="package://snp_automate_2023/meshes/collision/ati_standoff.ply"/>
       </geometry>
     </collision>
     <collision>
       <geometry>
-        <mesh filename="package://snp_automate_2023/meshes/hc10_standoff.ply"/>
+        <mesh filename="package://snp_automate_2023/meshes/collision/hc10_standoff.ply"/>
       </geometry>
     </collision>
     <collision>
       <geometry>
-        <mesh filename="package://snp_automate_2023/meshes/sensor_bracket.ply"/>
+        <mesh filename="package://snp_automate_2023/meshes/collision/sensor_bracket.ply"/>
       </geometry>
     </collision>
     <collision>
       <geometry>
-        <mesh filename="package://snp_automate_2023/meshes/sponge.ply"/>
+        <mesh filename="package://snp_automate_2023/meshes/collision/sponge.ply"/>
       </geometry>
     </collision>

Commit message: Load YAML in xacro with support for older distros

File: snp_automate_2023/urdf/workcell.xacro (robot description, xacro)
@@ -165,5 +165,11 @@
     <origin rpy="0.0 0.0 ${radians(45)}"/>
   </joint>
-  <xacro:property name="camera_cal" value="${xacro.load_yaml('$(find snp_automate_2023)/config/calibration.yaml')}" />
+  <xacro:arg name="ros_distro" default="humble"/>
+  <xacro:if value="${'$(arg ros_distro)' > 'foxy'}">
+    <xacro:property name="camera_cal" value="${xacro.load_yaml('$(find snp_automate_2022)/config/camera_calibration.yaml')}" />
+  </xacro:if>
+  <xacro:unless value="${'$(arg ros_distro)' > 'foxy'}">
+    <xacro:property name="camera_cal" value="${load_yaml('$(find snp_automate_2022)/config/camera_calibration.yaml')}" />
+  </xacro:unless>
   <link name="camera_color_optical_frame"/>
   <joint name="tool0_to_camera" type="fixed">

Commit message: fix config filepath typos in launch file

File: snp_automate_2023/urdf/workcell.xacro (robot description, xacro)
@@ -167,8 +167,8 @@
   <xacro:arg name="ros_distro" default="humble"/>
   <xacro:if value="${'$(arg ros_distro)' > 'foxy'}">
-    <xacro:property name="camera_cal" value="${xacro.load_yaml('$(find snp_automate_2022)/config/camera_calibration.yaml')}" />
+    <xacro:property name="camera_cal" value="${xacro.load_yaml('$(find snp_automate_2023)/config/calibration.yaml')}" />
   </xacro:if>
   <xacro:unless value="${'$(arg ros_distro)' > 'foxy'}">
-    <xacro:property name="camera_cal" value="${load_yaml('$(find snp_automate_2022)/config/camera_calibration.yaml')}" />
+    <xacro:property name="camera_cal" value="${load_yaml('$(find snp_automate_2023)/config/calibration.yaml')}" />
   </xacro:unless>
   <link name="camera_color_optical_frame"/>
